File: Pcb/MBoard_One_Stm32H734_KiCad_project/MBoard_One_Stm32H734_KiCad_project.sch (KiCad schematic (older format))
At the start: 17 parts

Commit message: Auto stash before merge of "MB100-PCB-developing" and "origin/MB100-PCB-developing"
Parts:
- removed U?: FT232H, symbol Interface_USB:FT232H
- gave numbers to parts that had none: 1
Other:
- moved on the sheet: U1
Changed lines of the file:
@@
 EESchema Schematic File Version 4
+LIBS:MBoard_One_Stm32H734_KiCad_project-cache
 EELAYER 26 0
 EELAYER END
@@
 $EndDescr
 $Comp
-L MCU_ST_STM32H7:STM32H743ZITx U?
+L MCU_ST_STM32H7:STM32H743ZITx U1
 U 1 1 5C5D4170
-P 10800 8350
-F 0 "U?" H 10750 4664 50  0000 C CNN
-F 1 "STM32H743ZITx" H 10750 4573 50  0000 C CNN
-F 2 "Package_QFP:LQFP-144_20x20mm_P0.5mm" H 9700 4950 50  0001 R CNN
-F 3 "http://www.st.com/st-web-ui/static/active/en/resource/technical/document/datasheet/DM00387108.pdf" H 10800 8350 50  0001 C CNN
-	1    10800 8350
+P 10650 8250
+F 0 "U1" H 10600 4564 50  0000 C CNN
+F 1 "STM32H743ZITx" H 10600 4473 50  0000 C CNN
+F 2 "Package_QFP:LQFP-144_20x20mm_P0.5mm" H 9550 4850 50  0001 C CNN
+F 3 "http://www.st.com/st-web-ui/static/active/en/resource/technical/document/datasheet/DM00387108.pdf" H 10650 8250 50  0001 C CNN
+	1    10650 8250
 	1    0    0    -1
 $EndComp
@@
 F 3 "http://www.ti.com/lit/ds/symlink/pcm5102.pdf" H 19900 6300 50  0001 C CNN
 	1    19950 5550
-	1    0    0    -1
-$EndComp
-$Comp
-L Interface_USB:FT232H U?
-U 1 1 5C5D445B
-P 19950 8550
-F 0 "U?" H 19950 10228 50  0000 C CNN
-F 1 "FT232H" H 19950 10137 50  0000 C CNN
-F 2 "" H 19950 8550 50  0001 C CNN
-F 3 "http://www.ftdichip.com/Products/ICs/FT232H.htm" H 19950 8550 50  0001 C CNN
-	1    19950 8550
 	1    0    0    -1
 $EndComp
@@
 	1    0    0    -1
 $EndComp
+$Comp
+L power:GNDREF #PWR?
+U 1 1 5C63FC76
+P 11700 11900
+F 0 "#PWR?" H 11700 11650 50  0001 C CNN
+F 1 "GNDREF" H 11705 11727 50  0000 C CNN
+F 2 "" H 11700 11900 50  0001 C CNN
+F 3 "" H 11700 11900 50  0001 C CNN
+	1    11700 11900
+	1    0    0    -1
+$EndComp
+$Comp
+L power:GNDA #PWR?
+U 1 1 5C64065A
+P 11700 12250
+F 0 "#PWR?" H 11700 12000 50  0001 C CNN
+F 1 "GNDA" H 11705 12077 50  0000 C CNN
+F 2 "" H 11700 12250 50  0001 C CNN
+F 3 "" H 11700 12250 50  0001 C CNN
+	1    11700 12250
+	1    0    0    -1
+$EndComp

Commit message: Updating to the PCB
Parts:
- removed U1: STM32H743ZITx, Package_QFP:LQFP-144_20x20mm_P0.5mm, symbol MCU_ST_STM32H7:STM32H743ZITx
- removed U?: AT25SF081-SSHD-X, Package_SO:SOIC-8_3.9x4.9mm_P1.27mm, symbol Memory_Flash:AT25SF081-SSHD-X
- removed U?: VL53L0X, SENSOR_VL53L0X, symbol VL53L0X:VL53L0X
- added C? (x3): 100nF, symbol Device:C
- added C?: 1uF, symbol Device:C
- added C?: 1nF, symbol Device:C
- added C? (x4): 0.1uF, symbol Device:C
- added C?: C, symbol Device:C
- added D?: DIODE, symbol pspice:DIODE
- added R, R?: 100kOhm, symbol Device:R
- added R? (x4): 4.7kOhm, symbol Device:R
- added R?: 1kOhm, symbol Device:R
- added R?: 100kOm, symbol Device:R
- added R? (x12): 10kOhm, symbol Device:R
- added R? (x2): 3.3kOhm, symbol Device:R
- added TH?: 10kOhm, symbol Device:Thermistor_NTC
- added U1: STM32H743BITx, Package_QFP:LQFP-208_28x28mm_P0.5mm, symbol MCU_ST_STM32H7:STM32H743BITx
- added U?: MT28EW01GABA1LPC-0SIT_TR, BGA64C100P8X8_1300X1100X130N, symbol MT28EW01GABA1LPC-0SIT_TR:MT28EW01GABA1LPC-0SIT_TR
- added U?: MT48LC16M16A2TG-6A_IT_GTR, SOP80P1176X120-54N, symbol MT48LC16M16A2TG-6A_IT_GTR:MT48LC16M16A2TG-6A_IT_GTR
- added U?: VL53L0X, SENSOR_VL53L0X, symbol VL53L0X:VL53L0X
Connections:
- net GNDREF: now also U?.1 (GND), U?.7 (GND)
- net +3V3: now reaches U?.2 (CSB)
- net +3V3: now also IC?.7 (VDD), U?.1 (RESV_VDDIO), U?.1 (VCC), U?.13 (VDD), U?.2 (ADDR), U?.6 (VDD), U?.6 (VDDIO), U?.8 (VCC), U?.8 (VDD), U?.8 (VDDIO), C?.1, C?.1, C?.1, C?.1, C?.1, C?.1, R.1, R?.1, R?.1, R?.1, R?.1, R?.1, R?.1, R?.1, R?.1, R?.1, R?.1, R?.1, R?.1
- net MCU_I2C0_SDA: now reaches U?.3 (SDI)
- net MCU_I2C0_SDA: now also U?.24 (SDA/MOSI), U?.4 (SDA), U?.9 (SDA), R?.2, R?.2
- net MCU_I2C0_SCL: now reaches U?.4 (SCK)
- net MCU_I2C0_SCL: now also U?.10 (SCL), U?.23 (SCL/SCLK), U?.6 (SCL), R?.2, R?.2
- net GNDD: now reaches U?.5 (SDO)
- net GNDD: now also IC?.5 (GND), U?.11 (GND), U?.11 (GPIO9), U?.12 (GND), U?.12 (GPIO10), U?.15 (GND), U?.18 (GND), U?.19 (GPIO4), U?.2 (AVSSVCSEL), U?.20 (GPIO5), U?.20 (RESV_GND), U?.3 (GND), U?.3 (GND), U?.4 (GND), U?.4 (GPIO16), U?.5 (GPIO14), U?.6 (GND), U?.6 (GPIO12), U?.7 (GPIO13), C?.2, C?.2, C?.2, C?.2, C?.2, C?.2, C?.2, C?.2, C?.2, C?.2, R?.2, R?.2, R?.2, R?.2, R?.2, U?.12 (GND), U?.2 (AVSSVCSEL), U?.3 (GND), U?.4 (GND), U?.6 (GND)
- net at U?.1 (ADDR): now also R?.1
- net SCL: now reaches U?.10 (SCL)
- net at U?.2 (~RESET): now also D?.1 (K)
- net MCU_CCS_INT_GPIO_PIN: now reaches U?.3 (~INT)
- net at U?.4 (PWM): now also U?.5 (Sense), TH?.1
- net at U?.7 (~WAKE): now also R?.2
- net at U?.8 (AUX): now also R.2, TH?.2
- net SDA: now reaches U?.9 (SDA)
- net at U?.10 (REGOUT): now also C?.1
- net at U?.11 (FSYNC): now also R?.1
- net MCU_MPU_INT_GPIO_PIN: now reaches U?.12 (INT)
- net at U?.22 (~CS): now also R?.2
- net at U?.9 (AD0/MISO): now also R?.1
- net at U?.5 (DVI): now also R?.2
- net MCU_ESP_RST_GPIO_PIN: now reaches U?.1 (~RST)
- net MCU_ESP_RST_GPIO_PIN: now also R?.2
- net at U?.10 (MISO): now also U?.13 (MOSI), U?.14 (SCLK), R?.1
- net at U?.16 (GPIO15): now also R?.1
- net at U?.17 (GPIO2): now also R?.2
- net at U?.18 (GPIO0): now also R?.2
- net MCU_ESP_USART_TXD: now reaches U?.21 (GPIO3/RXD)
- net MCU_ESP_USART_RXD: now reaches U?.22 (GPIO1/TXD)
- net MCU_ESP_EN_GPIO_PIN: now reaches U?.3 (EN)
- net MCU_ESP_EN_GPIO_PIN: now also R?.2
- net at U?.9 (CS0): now also R?.2
- net +2V8: now reaches U?.1 (AVDDVCSEL)
- net +2V8: now also U?.11 (AVDD), C?.1, C?.1, R?.1, R?.1, R?.1, R?.1, U?.1 (AVDDVCSEL), U?.11 (AVDD)
- net at U?.5 (~XSHUT~): now also R?.2
- net at U?.7 (GPIO1): now also R?.2
- net at IC?.10 (TR): now also C?.1
- net MCU_ML_EN_GPIO_PIN: now reaches IC?.4 (EN)
- net MCU_ML_OUT_ADC: now reaches IC?.8 (OUT)
- new net: U?.D8 (VCCQ), U?.F1 (VCCQ)
- new net: U?.E8 (VSS), U?.H2 (VSS), U?.H7 (VSS)
- new net: U?.1 (VDD), U?.14 (VDD), U?.27 (VDD)
- new net: U?.12 (VSSQ), U?.46 (VSSQ), U?.52 (VSSQ), U?.6 (VSSQ)
- new net: U?.28 (VSS), U?.41 (VSS), U?.54 (VSS)
- new net: U?.3 (VDDQ), U?.43 (VDDQ), U?.49 (VDDQ), U?.9 (VDDQ)
- new net: R?.2, U?.5 (~XSHUT~)
- new net: R?.2, U?.7 (GPIO1)
- new net MCU_CCS_RST_GPIO_PIN: D?.2 (A)
- new net MCU_I2C1_SCL: U?.10 (SCL)
- new net MCU_I2C1_SDA: U?.9 (SDA)
- no-connect marks 0 -> 10
Other:
- note added: "Don't forget that only for one I2C bus can be SDA & SCL resistors.\nAnd the values must be every 4.7 kOhm."
- moved on the sheet: IC?, U?

Commit message: Continuing PCB develop
Parts:
- added J?: SD_Card, symbol Connector:SD_Card
Connections:
- net +3V3: now also U1.103 (VDD), U1.115 (VDD), U1.124 (VDD), U1.15 (VDD), U1.150 (VDD), U1.158 (VDD), U1.171 (VDD), U1.185 (VDD), U1.204 (VDD), U1.26 (VDD), U1.39 (VDD), U1.52 (VDD), U1.59 (VDD), U1.73 (VDD), U1.83 (VDD), U1.94 (VDD)
- net MCU_I2C0_SCL: now also U1.198 (PB8)
- net MCU_I2C0_SDA: now also U1.196 (PB7)
Other:
- moved on the sheet: U?
Changed lines of the file:
@@
 L INA219:INA219 U?
 U 1 1 5C5D518D
-P 20700 2000
-F 0 "U?" H 20700 2867 50  0000 C CNN
-F 1 "INA219" H 20700 2776 50  0000 C CNN
-F 2 "SOT23-8" H 20700 2000 50  0001 L BNN
-F 3 "INA219" H 20700 2000 50  0001 L BNN
-F 4 "None" H 20700 2000 50  0001 L BNN "Field4"
-F 5 "Texas Instruments" H 20700 2000 50  0001 L BNN "Field5"
-F 6 "None" H 20700 2000 50  0001 L BNN "Field6"
-F 7 "Unavailable" H 20700 2000 50  0001 L BNN "Field7"
-F 8 "the ina219 is a high-side current shunt and power monitor with an i2c interface. the ina219 monitors both shunt drop ..." H 20700 2000 50  0001 L BNN "Field8"
-	1    20700 2000
+P 19950 1800
+F 0 "U?" H 19950 2667 50  0000 C CNN
+F 1 "INA219" H 19950 2576 50  0000 C CNN
+F 2 "SOT23-8" H 19950 1800 50  0001 L BNN
+F 3 "INA219" H 19950 1800 50  0001 L BNN
+F 4 "None" H 19950 1800 50  0001 L BNN "Field4"
+F 5 "Texas Instruments" H 19950 1800 50  0001 L BNN "Field5"
+F 6 "None" H 19950 1800 50  0001 L BNN "Field6"
+F 7 "Unavailable" H 19950 1800 50  0001 L BNN "Field7"
+F 8 "the ina219 is a high-side current shunt and power monitor with an i2c interface. the ina219 monitors both shunt drop ..." H 19950 1800 50  0001 L BNN "Field8"
+	1    19950 1800
 	1    0    0    -1
 $EndComp
@@
 L F-3188_CSR8645:F-3188_CSR8645 U?
 U 1 1 5C5D6029
-P 11300 3200
-F 0 "U?" H 11100 5037 60  0000 C CNN
-F 1 "F-3188_CSR8645" H 11100 4931 60  0000 C CNN
-F 2 "" H 11300 1500 60  0000 C CNN
-F 3 "" H 11300 1500 60  0000 C CNN
-	1    11300 3200
+P 5550 3350
+F 0 "U?" H 5350 5187 60  0000 C CNN
+F 1 "F-3188_CSR8645" H 5350 5081 60  0000 C CNN
+F 2 "" H 5550 1650 60  0000 C CNN
+F 3 "" H 5550 1650 60  0000 C CNN
+	1    5550 3350
 	1    0    0    -1
 $EndComp
@@
 Wire Wire Line
 	13300 7600 13150 7600
+$Comp
+L Connector:SD_Card J?
+U 1 1 5C7E5DE7
+P 1850 2700
+F 0 "J?" H 1850 3365 50  0000 C CNN
+F 1 "SD_Card" H 1850 3274 50  0000 C CNN
+F 2 "" H 1850 2700 50  0001 C CNN
+F 3 "http://portal.fciconnect.com/Comergent//fci/drawing/10067847.pdf" H 1850 2700 50  0001 C CNN
+	1    1850 2700
+	1    0    0    -1
+$EndComp
+$Comp
+L power:+3V3 #PWR?
+U 1 1 5C8092B6
+P 9500 3100
+F 0 "#PWR?" H 9500 2950 50  0001 C CNN
+F 1 "+3V3" H 9515 3273 50  0000 C CNN
+F 2 "" H 9500 3100 50  0001 C CNN
+F 3 "" H 9500 3100 50  0001 C CNN
+	1    9500 3100
+	1    0    0    -1
+$EndComp
+Wire Wire Line
+	7800 3650 7800 3200
+Wire Wire Line
+	7800 3200 7900 3200
+Wire Wire Line
+	9500 3200 9500 3100
+Wire Wire Line
+	7900 3650 7900 3200
+Connection ~ 7900 3200
+Wire Wire Line
+	7900 3200 8000 3200
+Wire Wire Line
+	8000 3650 8000 3200
+Connection ~ 8000 3200
+Wire Wire Line
+	8000 3200 8100 3200
+Wire Wire Line
+	8100 3650 8100 3200
+Connection ~ 8100 3200
+Wire Wire Line
+	8100 3200 8200 3200
+Wire Wire Line
+	8200 3650 8200 3200
+Connection ~ 8200 3200
+Wire Wire Line
+	8200 3200 8300 3200
+Wire Wire Line
+	8300 3650 8300 3200
+Connection ~ 8300 3200
+Wire Wire Line
+	8400 3650 8400 3200
+Wire Wire Line
+	8300 3200 8400 3200
+Connection ~ 8400 3200
+Wire Wire Line
+	8500 3650 8500 3200
+Wire Wire Line
+	8400 3200 8500 3200
+Connection ~ 8500 3200
+Wire Wire Line
+	8500 3200 8600 3200
+Wire Wire Line
+	8600 3650 8600 3200
+Connection ~ 8600 3200
+Wire Wire Line
+	8600 3200 8700 3200
+Wire Wire Line
+	8700 3650 8700 3200
+Connection ~ 8700 3200
+Wire Wire Line
+	8700 3200 8800 3200
+Wire Wire Line
+	8800 3650 8800 3200
+Connection ~ 8800 3200
+Wire Wire Line
+	8800 3200 8900 3200
+Connection ~ 8900 3200
+Wire Wire Line
+	8900 3200 9000 3200
+Wire Wire Line
+	9000 3650 9000 3200
+Connection ~ 9000 3200
+Wire Wire Line
+	9000 3200 9100 3200
+Wire Wire Line
+	8900 3200 8900 3650
+Wire Wire Line
+	9100 3650 9100 3200
+Connection ~ 9100 3200
+Wire Wire Line
+	9100 3200 9200 3200
+Wire Wire Line
+	9200 3650 9200 3200
+Connection ~ 9200 3200
+Wire Wire Line
+	9200 3200 9300 3200
+Wire Wire Line
+	9300 3650 9300 3200
+Connection ~ 9300 3200
+Wire Wire Line
+	9300 3200 9500 3200
+Text GLabel 10750 6450 2    50   Input ~ 0
+MCU_I2C0_SCL
+Text GLabel 10750 6350 2    50   Input ~ 0
+MCU_I2C0_SDA
+Wire Wire Line
+	10750 6350 10100 6350
+Wire Wire Line
+	10750 6450 10100 6450
 $EndSCHEMATC
